File: board_top_L/top_L.kicad_pcb (KiCad board)
At the start: 2 copper layers, 275 x 230 mm, 137 parts, among them J1 USB_C_Receptacle_USB2.0, J2 USB_C_Receptacle_USB2.0, P1 USB_C_Plug, Q1 MMBT5551L, Q10 MMBT5551L, Q11 MMBT5551L, Q12 MMBT5551L, Q13 MMBT5551L, Q14 MMBT5551L, Q2 MMBT5551L, Q3 MMBT5551L, Q4 MMBT5551L, Q5 MMBT5551L, Q6 MMBT5551L, Q7 MMBT5551L, Q8 MMBT5551L, Q9 MMBT5551L, SW1 Reset, SW2 Next, SW3 Previous, SW4 boot, SW5 run, U1 AP2112K-3.3, U2 W25Q128JVS, U3 RP2040, U4 SM420561N, U5 SM420561N, U6 SM420561N, U7 SM420561N, U8 SN74AHCT125QDRG4Q1, U9 PCF8591, Y1 ABLS-12.000MHZ-B4-T

Commit message: added BoM
Parts:
- Y1: footprint Crystal:Crystal_SMD_3225-4Pin_3.2x2.5mm -> Crystal:Crystal_SMD_2520-4Pin_2.5x2.0mm
Changed lines of the file:
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@@
     )
   )
-  (footprint "Crystal:Crystal_SMD_3225-4Pin_3.2x2.5mm" (layer "B.Cu")
+  (footprint "Crystal:Crystal_SMD_2520-4Pin_2.5x2.0mm" (layer "B.Cu")
     (at 83.9 178.8 180)
-    (descr "SMD Crystal SERIES SMD3225/4 http://www.txccrystal.com/images/pdf/7m-accuracy.pdf, 3.2x2.5mm^2 package")
+    (descr "SMD Crystal SERIES SMD2520/4 http://www.newxtal.com/UploadFiles/Images/2012-11-12-09-29-09-776.pdf, 2.5x2.0mm^2 package")
     (tags "SMD SMT crystal")
     (property "Sheetfile" "top_L.kicad_sch")
     (property "Sheetname" "")
     (attr smd)
-    (fp_text reference "Y1" (at 0 -2.45) (layer "B.SilkS")
+    (fp_text reference "Y1" (at 0 2.2) (layer "B.SilkS")
       (effects (font (size 1 1) (thickness 0.15)) (justify mirror))
     )
-    (fp_text value "ABLS-12.000MHZ-B4-T" (at 0 -2.45) (layer "B.Fab")
+    (fp_text value "ABLS-12.000MHZ-B4-T" (at 0 -2.2) (layer "B.Fab")
       (effects (font (size 1 1) (thickness 0.15)) (justify mirror))
     )
     (fp_text user "${REFERENCE}" (at 0 0) (layer "B.Fab")
-      (effects (font (size 0.7 0.7) (thickness 0.105)) (justify mirror))
+      (effects (font (size 0.6 0.6) (thickness 0.09)) (justify mirror))
     )
-    (fp_line (start -2 1.65) (end -2 -1.65) (layer "B.SilkS") (width 0.12))
-    (fp_line (start -2 -1.65) (end 2 -1.65) (layer "B.SilkS") (width 0.12))
-    (fp_line (start -2.1 1.7) (end -2.1 -1.7) (layer "B.CrtYd") (width 0.05))
-    (fp_line (start 2.1 1.7) (end -2.1 1.7) (layer "B.CrtYd") (width 0.05))
-    (fp_line (start 2.1 -1.7) (end 2.1 1.7) (layer "B.CrtYd") (width 0.05))
-    (fp_line (start -2.1 -1.7) (end 2.1 -1.7) (layer "B.CrtYd") (width 0.05))
-    (fp_line (start 1.6 1.25) (end -1.6 1.25) (layer "B.Fab") (width 0.1))
-    (fp_line (start -1.6 1.25) (end -1.6 -1.25) (layer "B.Fab") (width 0.1))
-    (fp_line (start 1.6 -1.25) (end 1.6 1.25) (layer "B.Fab") (width 0.1))
-    (fp_line (start -1.6 -0.25) (end -0.6 -1.25) (layer "B.Fab") (width 0.1))
-    (fp_line (start -1.6 -1.25) (end 1.6 -1.25) (layer "B.Fab") (width 0.1))
-    (pad "1" smd rect (at -1.1 -0.85 180) (size 1.4 1.2) (layers "B.Cu" "B.Paste" "B.Mask")
+    (fp_line (start -1.65 -1.4) (end 1.65 -1.4) (layer "B.SilkS") (width 0.12))
+    (fp_line (start -1.65 1.4) (end -1.65 -1.4) (layer "B.SilkS") (width 0.12))
+    (fp_line (start -1.7 1.5) (end -1.7 -1.5) (layer "B.CrtYd") (width 0.05))
+    (fp_line (start 1.7 1.5) (end -1.7 1.5) (layer "B.CrtYd") (width 0.05))
+    (fp_line (start -1.7 -1.5) (end 1.7 -1.5) (layer "B.CrtYd") (width 0.05))
+    (fp_line (start 1.7 -1.5) (end 1.7 1.5) (layer "B.CrtYd") (width 0.05))
+    (fp_line (start -1.15 -1) (end -1.25 -0.9) (layer "B.Fab") (width 0.1))
+    (fp_line (start 1.25 -0.9) (end 1.15 -1) (layer "B.Fab") (width 0.1))
+    (fp_line (start -1.25 0) (end -0.25 -1) (layer "B.Fab") (width 0.1))
+    (fp_line (start -1.15 1) (end 1.15 1) (layer "B.Fab") (width 0.1))
+    (fp_line (start 1.15 -1) (end -1.15 -1) (layer "B.Fab") (width 0.1))
+    (fp_line (start 1.15 1) (end 1.25 0.9) (layer "B.Fab") (width 0.1))
+    (fp_line (start 1.25 0.9) (end 1.25 -0.9) (layer "B.Fab") (width 0.1))
+    (fp_line (start -1.25 0.9) (end -1.15 1) (layer "B.Fab") (width 0.1))
+    (fp_line (start -1.25 -0.9) (end -1.25 0.9) (layer "B.Fab") (width 0.1))
+    (pad "1" smd rect (at -0.875 -0.7 180) (size 1.15 1) (layers "B.Cu" "B.Paste" "B.Mask")
       (net 6 "/XIN") (pinfunction "1") (pintype "passive"))
-    (pad "2" smd rect (at 1.1 -0.85 180) (size 1.4 1.2) (layers "B.Cu" "B.Paste" "B.Mask")
+    (pad "2" smd rect (at 0.875 -0.7 180) (size 1.15 1) (layers "B.Cu" "B.Paste" "B.Mask")
       (net 2 "GND") (pinfunction "2") (pintype "passive"))
-    (pad "3" smd rect (at 1.1 0.85 180) (size 1.4 1.2) (layers "B.Cu" "B.Paste" "B.Mask")
+    (pad "3" smd rect (at 0.875 0.7 180) (size 1.15 1) (layers "B.Cu" "B.Paste" "B.Mask")
       (net 7 "Net-(C20-Pad1)") (pinfunction "3") (pintype "passive"))
-    (pad "4" smd rect (at -1.1 0.85 180) (size 1.4 1.2) (layers "B.Cu" "B.Paste" "B.Mask")
+    (pad "4" smd rect (at -0.875 0.7 180) (size 1.15 1) (layers "B.Cu" "B.Paste" "B.Mask")
       (net 2 "GND") (pinfunction "4") (pintype "passive"))
-    (model "${KICAD6_3DMODEL_DIR}/Crystal.3dshapes/Crystal_SMD_3225-4Pin_3.2x2.5mm.wrl"
+    (model "${KICAD6_3DMODEL_DIR}/Crystal.3dshapes/Crystal_SMD_2520-4Pin_2.5x2.0mm.wrl"
       (offset (xyz 0 0 0))
       (scale (xyz 1 1 1))
